File: Hardware Design/ProjectorController.brd (EAGLE design)
At the start: 39 x 34.9 mm, 18 parts, among them J1 5747844-4, J2 Cap Buttons, J3 Prog, J4 Prog/Run, J5 10118194-0001LF, U1 ESP-WROOM-32, U2 SP3232EEN-L

Commit message: PC-16 and other fixes
Routing:
- net N$6: track 7.42 -> 6.47 mm
- net GND: track 44.2 -> 43.7 mm
Changed lines of the file:
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@@
 </polygon>
 <wire x1="6.855" y1="56.639" x2="6.855" y2="55.499" width="0.1524" layer="16"/>
-<wire x1="8.542" y1="46.96" x2="9.174" y2="46.96" width="0.1524" layer="1"/>
+<wire x1="8.796" y1="46.96" x2="9.174" y2="46.96" width="0.1524" layer="1"/>
 <wire x1="6.132" y1="56.0176" x2="6.0706" y2="55.9562" width="0.1524" layer="1"/>
 <via x="6.35" y="57.658" extent="1-16" drill="0.35"/>
-<wire x1="16.4" y1="45.085" x2="20.32" y2="45.085" width="0.1524" layer="1"/>
-<wire x1="20.32" y1="45.085" x2="34.4" y2="45.085" width="0.1524" layer="1"/>
+<wire x1="16.019" y1="45.085" x2="20.32" y2="45.085" width="0.1524" layer="1"/>
+<wire x1="20.32" y1="45.085" x2="34.781" y2="45.085" width="0.1524" layer="1"/>
 <wire x1="26.1" y1="52.495" x2="20.32" y2="46.715" width="0.1524" layer="1"/>
 <wire x1="20.32" y1="46.715" x2="20.32" y2="45.085" width="0.1524" layer="1"/>
 <wire x1="35.27" y1="48.095" x2="35.27" y2="45.955" width="0.1524" layer="16"/>
-<wire x1="16.4" y1="45.085" x2="13.335" y2="45.085" width="0.1524" layer="1"/>
+<wire x1="16.019" y1="45.085" x2="13.335" y2="45.085" width="0.1524" layer="1"/>
 <wire x1="13.335" y1="45.085" x2="12.7" y2="45.72" width="0.1524" layer="1"/>
 <wire x1="13.465" y1="61.973" x2="13.462" y2="61.976" width="0.1524" layer="1"/>
 <wire x1="30.48" y1="64.77" x2="31.115" y2="64.135" width="0.1524" layer="1"/>
-<wire x1="31.115" y1="64.135" x2="31.115" y2="63.095" width="0.1524" layer="1"/>
+<wire x1="31.115" y1="64.135" x2="31.115" y2="63.476" width="0.1524" layer="1"/>
 <via x="30.48" y="64.77" extent="1-16" drill="0.35"/>
-<wire x1="8.542" y1="46.96" x2="11.46" y2="46.96" width="0.1524" layer="1"/>
+<wire x1="8.796" y1="46.96" x2="11.46" y2="46.96" width="0.1524" layer="1"/>
 <wire x1="11.46" y1="46.96" x2="12.7" y2="45.72" width="0.1524" layer="1"/>
 <wire x1="6.0706" y1="55.9562" x2="6.0706" y2="57.3786" width="0.1524" layer="1"/>
@@
 <contactref element="U2" pad="16"/>
 <contactref element="C3" pad="2"/>
-<wire x1="9.655" y1="56.128" x2="9.655" y2="55.499" width="0.1524" layer="16"/>
 <wire x1="12.7" y1="53.34" x2="11.814" y2="53.34" width="0.1524" layer="16"/>
 <via x="33.02" y="46.99" extent="1-16" drill="0.35"/>
 <wire x1="33.02" y1="46.99" x2="33.655" y2="46.355" width="0.1524" layer="1"/>
-<wire x1="33.655" y1="46.355" x2="34.4" y2="46.355" width="0.1524" layer="1"/>
+<wire x1="33.655" y1="46.355" x2="34.781" y2="46.355" width="0.1524" layer="1"/>
 <wire x1="30.477" y1="46.99" x2="30.4785" y2="46.9885" width="0.1524" layer="16"/>
 <wire x1="33.02" y1="46.99" x2="33.0185" y2="46.9885" width="0.1524" layer="16"/>
@@
 <contactref element="J5" pad="1"/>
 <wire x1="10.665" y1="55.9278" x2="10.6934" y2="55.9562" width="0.1524" layer="1"/>
-<wire x1="8.542" y1="49.56" x2="8.572" y2="49.53" width="0.1524" layer="1"/>
 <wire x1="9.655" y1="60.325" x2="9.655" y2="60.195" width="0.1524" layer="16"/>
 <wire x1="12.065" y1="57.785" x2="9.655" y2="60.195" width="0.1524" layer="16"/>
@@
 <wire x1="10.13" y1="49.56" x2="10.665" y2="50.095" width="0.1524" layer="1"/>
 <wire x1="10.665" y1="50.095" x2="10.665" y2="55.9278" width="0.1524" layer="1"/>
+<wire x1="8.542" y1="49.56" x2="8.763" y2="49.56" width="0" layer="19" extent="1-1"/>
 </signal>
 <signal name="N$1">
 <contactref element="U1" pad="23"/>
 <contactref element="J2" pad="3"/>
-<wire x1="39.893" y1="62.753" x2="40.005" y2="62.753" width="0.1524" layer="16"/>
 <wire x1="31.76865" y1="60.96" x2="33.38705" y2="62.5784" width="0.1524" layer="1"/>
 <wire x1="39.8304" y1="62.5784" x2="40.005" y2="62.753" width="0.1524" layer="1"/>
 <wire x1="33.38705" y1="62.5784" x2="39.8304" y2="62.5784" width="0.1524" layer="1"/>
-<wire x1="20.955" y1="62.79970625" x2="20.955" y2="63.095" width="0.1524" layer="1"/>
+<wire x1="20.955" y1="62.79970625" x2="20.955" y2="63.476" width="0.1524" layer="1"/>
 <wire x1="22.79470625" y1="60.96" x2="20.955" y2="62.79970625" width="0.1524" layer="1"/>
-<wire x1="31.76865" y1="60.96" x2="25.4" y2="60.96" width="0.1524" layer="1"/>
-<wire x1="25.4" y1="60.96" x2="22.79470625" y2="60.96" width="0.1524" layer="1"/>
+<wire x1="31.76865" y1="60.96" x2="22.79470625" y2="60.96" width="0.1524" layer="1"/>
 </signal>
 <signal name="N$2">
 <contactref element="U1" pad="9"/>
 <contactref element="J2" pad="1"/>
-<wire x1="34.4" y1="55.245" x2="34.9914" y2="55.8364" width="0.1524" layer="1"/>
+<wire x1="34.781" y1="55.245" x2="34.9914" y2="55.8364" width="0.1524" layer="1"/>
 <wire x1="40.005" y1="55.753" x2="39.9216" y2="55.8364" width="0.1524" layer="1"/>
 <wire x1="39.9216" y1="55.8364" x2="34.9914" y2="55.8364" width="0.1524" layer="1"/>
@@
 <contactref element="U1" pad="26"/>
 <contactref element="J2" pad="2"/>
-<wire x1="16.4" y1="60.325" x2="31.56470625" y2="60.325" width="0.1524" layer="1"/>
+<wire x1="16.019" y1="60.325" x2="31.56470625" y2="60.325" width="0.1524" layer="1"/>
 <wire x1="31.56470625" y1="60.325" x2="33.51330625" y2="62.2736" width="0.1524" layer="1"/>
 <wire x1="36.9844" y1="62.2736" x2="40.005" y2="59.253" width="0.1524" layer="1"/>
@@
 <contactref element="R1" pad="2"/>
 <contactref element="S1" pad="B2"/>
-<wire x1="34.4" y1="47.625" x2="33.655" y2="47.625" width="0.1524" layer="1"/>
+<wire x1="34.781" y1="47.625" x2="33.655" y2="47.625" width="0.1524" layer="1"/>
 <wire x1="33.655" y1="47.625" x2="33.02" y2="48.26" width="0.1524" layer="1"/>
 <via x="33.02" y="48.26" extent="1-16" drill="0.35"/>
@@
 <contactref element="U1" pad="25"/>
 <contactref element="R2" pad="2"/>
-<wire x1="16.4" y1="61.595" x2="17.145" y2="61.595" width="0.1524" layer="1"/>
+<wire x1="16.019" y1="61.595" x2="17.145" y2="61.595" width="0.1524" layer="1"/>
 <wire x1="17.145" y1="61.595" x2="17.78" y2="60.96" width="0.1524" layer="1"/>
 <via x="17.78" y="60.96" extent="1-16" drill="0.35"/>
@@
 <contactref element="R2" pad="1"/>
 <contactref element="J4" pad="2"/>
-<wire x1="13.462" y1="59.436" x2="14.39985" y2="63.5" width="0.1524" layer="16"/>
-<wire x1="14.39985" y1="63.5" x2="17.65" y2="63.5" width="0.1524" layer="16"/>
+<wire x1="16.51" y1="63.5" x2="17.65" y2="63.5" width="0.1524" layer="16"/>
+<wire x1="13.462" y1="59.436" x2="15.24" y2="61.214" width="0.1524" layer="16"/>
+<wire x1="15.24" y1="61.214" x2="15.24" y2="62.23" width="0.1524" layer="16"/>
+<wire x1="15.24" y1="62.23" x2="16.51" y2="63.5" width="0.1524" layer="16"/>
 </signal>
 <signal name="N$7">
@@
 <contactref element="J3" pad="2"/>
 <wire x1="12.7" y1="48.26" x2="13.335" y2="48.895" width="0.1524" layer="1"/>
-<wire x1="13.335" y1="48.895" x2="16.4" y2="48.895" width="0.1524" layer="1"/>
+<wire x1="13.335" y1="48.895" x2="16.019" y2="48.895" width="0.1524" layer="1"/>
 </signal>
 <signal name="N$8">
@@
 <wire x1="12.7" y1="50.8" x2="14.859" y2="50.8" width="0.1524" layer="1"/>
 <wire x1="14.859" y1="50.8" x2="15.494" y2="50.165" width="0.1524" layer="1"/>
-<wire x1="15.494" y1="50.165" x2="16.4" y2="50.165" width="0.1524" layer="1"/>
+<wire x1="15.494" y1="50.165" x2="16.019" y2="50.165" width="0.1524" layer="1"/>
 </signal>
 <signal name="N$10">
@@
 <contactref element="U2" pad="13"/>
 <contactref element="U1" pad="27"/>
-<wire x1="16.4" y1="59.055" x2="24.765" y2="59.055" width="0.1524" layer="1"/>
+<wire x1="16.019" y1="59.055" x2="24.765" y2="59.055" width="0.1524" layer="1"/>
 <via x="24.765" y="59.055" extent="1-16" drill="0.35"/>
 <wire x1="24.765" y1="60.7822" x2="24.765" y2="59.055" width="0.1524" layer="16"/>
@@
 <contactref element="U2" pad="11"/>
 <contactref element="U1" pad="28"/>
-<wire x1="22.225" y1="60.7822" x2="22.225" y2="60.325" width="0.1524" layer="16"/>
-<wire x1="16.4" y1="57.785" x2="22.225" y2="57.785" width="0.1524" layer="1"/>
+<wire x1="16.019" y1="57.785" x2="22.225" y2="57.785" width="0.1524" layer="1"/>
 <via x="22.225" y="57.785" extent="1-16" drill="0.35"/>
 <wire x1="22.225" y1="60.7822" x2="22.225" y2="57.785" width="0.1524" layer="16"/>
@@
 <contactref element="C5" pad="2"/>
 <contactref element="U2" pad="1"/>
-<wire x1="21.59" y1="49.4" x2="21.59" y2="49.53" width="0.1524" layer="16"/>
 <wire x1="21.59" y1="49.4" x2="22.86" y2="50.67" width="0.1524" layer="16"/>
 <wire x1="22.86" y1="50.67" x2="22.86" y2="50.8" width="0.1524" layer="16"/>
